File: 24x24 Matrix.kicad_pcb (KiCad board)
At the start: 4 copper layers, 55 x 63.4 mm, 599 parts, among them J1 Conn_01x06_Pin, J2 Conn_01x06_Pin, J3 SM06B-GHS-TB

Commit message: Added silkscreen and changed connector wiring
Connections:
- J3 pad 3: GND -> Block2
- J3 pad 4: Block2 -> Block1
- J3 pad 5: Block1 -> GND
Routing:
- net Block2: track 43.8 -> 50.3 mm
- net Block1: track 38.1 -> 41.1 mm
- net GND: track 1118.7 -> 1119.2 mm
- net Block3: track 39.8 -> 40.3 mm
Other:
- board text added: "5v"
- board text added: "GND"
